Commit message: Added more accurate collision model of kinect and set kinect publish rate to 30Hz

File: urdf/sensors/kinect.urdf.xacro (robot description, xacro)
@@ -31,7 +31,7 @@
       </visual>
   	  <collision>
-        <origin xyz="0.0 0.0 0.0" rpy="0 0 0"/>
+        <origin xyz="0.0478 0.0 0.0" rpy="0 0 -${M_PI/2}"/>
   	    <geometry>
-  	      <box size="0.07271 0.27794 0.073"/>
+  	      <mesh filename="package://turtlebot_description/meshes/sensors/kinect-collision.dae" scale="0.1 0.1 0.1"/>
   	    </geometry>
   	  </collision>

File: urdf/turtlebot_gazebo.urdf.xacro (robot description, xacro)
@@ -6,5 +6,5 @@
       <sensor type="depth" name="camera">
         <always_on>true</always_on>
-        <update_rate>20.0</update_rate>
+        <update_rate>30.0</update_rate>
         <camera>
           <horizontal_fov>${60.0*M_PI/180.0}</horizontal_fov>
@@ -22,5 +22,5 @@
           <cameraName>camera</cameraName>
           <alwaysOn>true</alwaysOn>
-          <updateRate>10</updateRate>
+          <updateRate>0</updateRate>
           <imageTopicName>rgb/image_raw</imageTopicName>
           <depthImageTopicName>depth/image_raw</depthImageTopicName>
